File: 8-Bit-CPU-main/kicad_files/8-bit cpu.kicad_pcb (KiCad board)
At the start: 4 copper layers, 173.5 x 115.5 mm, 97 parts, among them SW1 HX 3X4X2-2P-1.6N TACTILE SWIT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, U1 74HC173D,653, U10 74HC153D,653, U11 74HC153D,653, U12 74HC153D,653, U13 74HC245D,653, U14 74HC08D,653, U15 74HC08D,653, U16 74HC32D,653, U17 74HC32D,653, U18 74HC32D,653, U19 74HC32D,653, U2 74HC173D,653, U20 74HC04D,653, U21 74HC173D,653, U22 AT28C256-15SU, U23 AT28C256-15SU, U24 AT28C256-15SU, U25 SN74HC161DR, U26 SN74HC161DR, U27 SN74HC161DR, U28 SN74HC161DR, U29 SN74HC161DR, U3 74HC173D,653, U30 SN74HC161DR, U31 AT28C64B-15PU, U32 74HC173D,653, U33 74HC173D,653, U34 74HC173D,653, U35 74HC173D,653, U36 CD74HC283M96, U37 CD74HC283M96, U38 74HC153D,653, U39 74HC153D,653, U4 74HC173D,653, U40 74HC153D,653, U41 74HC153D,653, U42 74HC245D,653, U43 74HC139D,653, U44 74HC173D,653, U45 74HC173D,653, U46 74HC173D,653, U47 74HC173D,653, U48 74HC173D,653, U49 74HC173D,653, U5 CD74HC283M96, U50 74HC173D,653, U51 74HC173D,653, U52 SN74HC161DR, U53 SN74HC161DR, U54 SN74HC161DR, U55 74HC173D,653, U56 74HC173D,653, U57 AT28C256-15SU, U58 AT28C256-15SU, U59 AT28C256-15SU, U6 CD74HC283M96, U60 AT28C64B-15PU, U61 HM6116LP-4, U62 OT70501MJBA4SL, U63 SN74HC14DR, U7 SN74HC86DR, U8 SN74HC86DR, U9 74HC153D,653

Commit message: Add files via upload
Connections:
- net N_4952B58E renamed Net-(U63-1A)
- C1 pad 1: A13 -> +5V
- C1 pad 2: OSC_OE -> GND
- C10 pad 1: A13 -> +5V
- C10 pad 2: OSC_OE -> GND
- C11 pad 1: A13 -> +5V
- C11 pad 2: OSC_OE -> GND
- C12 pad 1: A13 -> +5V
- C12 pad 2: OSC_OE -> GND
- C13 pad 1: A13 -> +5V
- C13 pad 2: OSC_OE -> GND
- C14 pad 1: A13 -> +5V
- C14 pad 2: OSC_OE -> GND
- C15 pad 1: A13 -> +5V
- C15 pad 2: OSC_OE -> GND
- C16 pad 1: A13 -> +5V
- C16 pad 2: OSC_OE -> GND
- C17 pad 1: A13 -> +5V
- C17 pad 2: OSC_OE -> GND
- C18 pad 1: A13 -> +5V
- C18 pad 2: OSC_OE -> GND
- C19 pad 1: A13 -> +5V
- C19 pad 2: OSC_OE -> GND
- C2 pad 1: A13 -> +5V
- C2 pad 2: OSC_OE -> GND
- C20 pad 1: A13 -> +5V
- C20 pad 2: OSC_OE -> GND
- C21 pad 1: A13 -> +5V
- C21 pad 2: OSC_OE -> GND
- C22 pad 1: A13 -> +5V
- C22 pad 2: OSC_OE -> GND
- C23 pad 1: A13 -> +5V
- C23 pad 2: OSC_OE -> GND
- C24 pad 1: A13 -> +5V
- C24 pad 2: OSC_OE -> GND
- C25 pad 1: A13 -> +5V
- C25 pad 2: OSC_OE -> GND
- C26 pad 1: A13 -> +5V
- C26 pad 2: OSC_OE -> GND
- C27 pad 1: A13 -> +5V
- C27 pad 2: OSC_OE -> GND
- C28 pad 1: A13 -> +5V
- C28 pad 2: OSC_OE -> GND
- C29 pad 1: A13 -> +5V
- C29 pad 2: OSC_OE -> GND
- C3 pad 1: A13 -> +5V
- C3 pad 2: OSC_OE -> GND
- C30 pad 1: A13 -> +5V
- C30 pad 2: OSC_OE -> GND
- C31 pad 1: A13 -> +5V
- C31 pad 2: OSC_OE -> GND
- C32 pad 1: A13 -> +5V
- C32 pad 2: OSC_OE -> GND
- C4 pad 1: A13 -> +5V
- C4 pad 2: OSC_OE -> GND
- C5 pad 1: A13 -> +5V
- C5 pad 2: OSC_OE -> GND
- C6 pad 1: A13 -> +5V
- C6 pad 2: OSC_OE -> GND
- C7 pad 1: A13 -> +5V
- C7 pad 2: OSC_OE -> GND
- C8 pad 1: A13 -> +5V
- C8 pad 2: OSC_OE -> GND
- C9 pad 1: A13 -> +5V
- C9 pad 2: OSC_OE -> GND
- R1 pad 1: A13 -> +5V
- SW1 pad 2: OSC_OE -> GND
- U1 pad 1: N_917A5B02 -> GND
- U1 pad 10: N_359D8FB6 -> MAR_LOW_IN
- U1 pad 11: DBUS3_2 -> DBUS3
- U1 pad 12: DBUS2_2 -> DBUS2
- U1 pad 13: DBUS1_2 -> DBUS1
- U1 pad 14: DBUS0_2 -> DBUS0
- U1 pad 15: OSC_OE -> GND
- U1 pad 16: A13 -> +5V
- U1 pad 2: N_907A596F -> GND
- U1 pad 3: ALU_A0_2 -> MARL0
- U1 pad 4: ALU_A1_2 -> MARL1
- U1 pad 5: ALU_A2_2 -> MARL2
- U1 pad 6: ALU_A3_2 -> MARL3
- U1 pad 7: CLK_2 -> CLK
- U1 pad 8: OSC_OE -> GND
- U1 pad 9: N_997A679A -> MAR_LOW_IN
- U10 pad 1: N_2B05052C -> GND
- U10 pad 10: N_D4E70B14 -> +5V
- U10 pad 11: N_D5E70CA7 -> GND
- U10 pad 12: N_D6E70E3A -> unconnected-(U10-2I2-Pad12)
- U10 pad 13: N_D7E70FCD -> unconnected-(U10-2I3-Pad13)
- U10 pad 14: N_D0E704C8 -> ZT_G7
- U10 pad 15: N_D1E7065B -> GND
- U10 pad 16: A13 -> +5V
- U10 pad 2: N_2E0509E5 -> GND
- U10 pad 3: N_2D050852 -> unconnected-(U10-1I3-Pad3)
- U10 pad 4: N_28050073 -> unconnected-(U10-1I2-Pad4)
- U10 pad 5: N_2704FEE0 -> GND
- U10 pad 6: N_2A050399 -> +5V
- U10 pad 7: N_29050206 -> Z_COMPUTED
- U10 pad 8: OSC_OE -> GND
- U10 pad 9: N_330511C4 -> Z_COMPUTED
- U11 pad 1: N_4627D9EB -> GND
- U11 pad 10: N_4BBBF3C1 -> +5V
- U11 pad 11: N_4ABBF22E -> GND
- U11 pad 12: N_49BBF09B -> unconnected-(U11-2I2-Pad12)
- U11 pad 13: N_48BBEF08 -> unconnected-(U11-2I3-Pad13)
- U11 pad 14: N_4FBBFA0D -> FI_OR
- U11 pad 15: N_4EBBF87A -> GND
- U11 pad 16: A13 -> +5V
- U11 pad 2: N_4727DB7E -> GND
- U11 pad 3: N_4827DD11 -> unconnected-(U11-1I3-Pad3)
- U11 pad 4: N_4927DEA4 -> unconnected-(U11-1I2-Pad4)
- U11 pad 5: N_4A27E037 -> GND
- U11 pad 6: N_4B27E1CA -> +5V
- U11 pad 7: N_4C27E35D -> FI_LATCH_N
- U11 pad 8: OSC_OE -> GND
- U11 pad 9: N_3E27CD53 -> FI_LATCH_N
- U12 pad 1: N_D4B68EE2 -> GND
- U12 pad 10: N_AD62D496 -> +5V
- U12 pad 11: N_AE62D629 -> GND
- U12 pad 12: N_AB62D170 -> unconnected-(U12-2I2-Pad12)
- U12 pad 13: N_AC62D303 -> unconnected-(U12-2I3-Pad13)
- U12 pad 14: N_B162DAE2 -> EO
- U12 pad 15: N_B262DC75 -> GND
- U12 pad 16: A13 -> +5V
- U12 pad 2: N_D3B68D4F -> GND
- U12 pad 3: N_D2B68BBC -> unconnected-(U12-1I3-Pad3)
- U12 pad 4: N_D1B68A29 -> unconnected-(U12-1I2-Pad4)
- U12 pad 5: N_D0B68896 -> GND
- U12 pad 6: N_CFB68703 -> +5V
- U12 pad 7: N_CEB68570 -> EO_N
- U12 pad 8: OSC_OE -> GND
- U12 pad 9: N_DCB69B7A -> EO_N
- U13 pad 1: N_6FDA2D21 -> unconnected-(U13-DIR-Pad1)
- U13 pad 10: OSC_OE -> GND
- U13 pad 11: N_2474F030 -> unconnected-(U13-B7-Pad11)
- U13 pad 12: N_2774F4E9 -> unconnected-(U13-B6-Pad12)
- U13 pad 13: N_2674F356 -> unconnected-(U13-B5-Pad13)
- U13 pad 14: N_2974F80F -> unconnected-(U13-B4-Pad14)
- U13 pad 15: N_2874F67C -> unconnected-(U13-B3-Pad15)
- U13 pad 16: N_2B74FB35 -> unconnected-(U13-B2-Pad16)
- U13 pad 17: N_2A74F9A2 -> unconnected-(U13-B1-Pad17)
- U13 pad 18: N_2D74FE5B -> unconnected-(U13-B0-Pad18)
- U13 pad 19: N_2C74FCC8 -> unconnected-(U13-~{OE}-Pad19)
- U13 pad 20: A13 -> +5V
- U13 pad 6: N_70DA2EB4 -> unconnected-(U13-A4-Pad6)
- U13 pad 7: N_71DA3047 -> unconnected-(U13-A5-Pad7)
- U13 pad 8: N_66DA1EF6 -> unconnected-(U13-A6-Pad8)
- U13 pad 9: N_67DA2089 -> unconnected-(U13-A7-Pad9)
- U14 pad 1: N_D6150B60 -> ALU_A0
- U14 pad 10: N_5320CEF0 -> ALU_B2
- U14 pad 11: N_5420D083 -> ALU_AND3
- U14 pad 12: N_5520D216 -> ALU_A3
- U14 pad 13: N_5620D3A9 -> ALU_B3
- U14 pad 14: A13 -> +5V
- U14 pad 2: N_D9151019 -> ALU_B0
- U14 pad 3: N_D8150E86 -> ALU_AND0
- U14 pad 4: N_DB15133F -> ALU_A1
- U14 pad 5: N_DA1511AC -> ALU_B1
- U14 pad 6: N_DD151665 -> ALU_AND1
- U14 pad 7: OSC_OE -> GND
- U14 pad 8: N_DF15198B -> ALU_AND2
- U14 pad 9: N_DE1517F8 -> ALU_A2
- U15 pad 1: N_71D67A5F -> ALU_A4
- U15 pad 10: N_A3A2BCBD -> ALU_B6
- U15 pad 11: N_A2A2BB2A -> ALU_AND7
- U15 pad 12: N_A1A2B997 -> ALU_A7
- U15 pad 13: N_A0A2B804 -> ALU_B7
- U15 pad 14: A13 -> +5V
- U15 pad 2: N_72D67BF2 -> ALU_B4
- U15 pad 3: N_73D67D85 -> ALU_AND4
- U15 pad 4: N_6CD67280 -> ALU_A5
- U15 pad 5: N_6DD67413 -> ALU_B5
- U15 pad 6: N_6ED675A6 -> ALU_AND5
- U15 pad 7: OSC_OE -> GND
- U15 pad 8: N_78D68564 -> ALU_AND6
- U15 pad 9: N_79D686F7 -> ALU_A6
- U16 pad 1: N_801646F6 -> ALU_A0
- U16 pad 10: N_691169B2 -> ALU_B2
- U16 pad 11: N_6A116B45 -> ALU_OR3
- U16 pad 12: N_6711668C -> ALU_A3
- U16 pad 13: N_6811681F -> ALU_B3
- U16 pad 14: A13 -> +5V
- U16 pad 2: N_7F164563 -> ALU_B0
- U16 pad 3: N_7E1643D0 -> ALU_OR0
- U16 pad 4: N_85164ED5 -> ALU_A1
- U16 pad 5: N_84164D42 -> ALU_B1
- U16 pad 6: N_83164BAF -> ALU_OR1
- U16 pad 7: OSC_OE -> GND
- U16 pad 8: N_89165521 -> ALU_OR2
- U16 pad 9: N_8816538E -> ALU_A2
- U17 pad 1: N_9B391BB5 -> ALU_A4
- U17 pad 10: N_DFE6525F -> ALU_B6
- U17 pad 11: N_DEE650CC -> ALU_OR7
- U17 pad 12: N_E1E65585 -> ALU_A7
- U17 pad 13: N_E0E653F2 -> ALU_B7
- U17 pad 14: A13 -> +5V
- U17 pad 2: N_983916FC -> ALU_B4
- U17 pad 3: N_9939188F -> ALU_OR4
- U17 pad 4: N_963913D6 -> ALU_A5
- U17 pad 5: N_97391569 -> ALU_B5
- U17 pad 6: N_943910B0 -> ALU_OR5
- U17 pad 7: OSC_OE -> GND
- U17 pad 8: N_A23926BA -> ALU_OR6
- U17 pad 9: N_A339284D -> ALU_A6
- U18 pad 1: N_21C3DE34 -> ALU_MUX_OUT0
- U18 pad 10: N_2B56804C -> ALU_MUX_OUT5
- U18 pad 11: N_2C5681DF -> ZT_G4
- U18 pad 12: N_2D568372 -> ALU_MUX_OUT6
- U18 pad 13: N_2E568505 -> ALU_MUX_OUT7
- U18 pad 14: A13 -> +5V
- U18 pad 2: N_24C3E2ED -> ALU_MUX_OUT1
- U18 pad 3: N_23C3E15A -> ZT_G1
- U18 pad 4: N_1EC3D97B -> ALU_MUX_OUT2
- U18 pad 5: N_1DC3D7E8 -> ALU_MUX_OUT3
- U18 pad 6: N_20C3DCA1 -> ZT_G2
- U18 pad 7: OSC_OE -> GND
- U18 pad 8: N_1AC3D32F -> ZT_G3
- U18 pad 9: N_19C3D19C -> ALU_MUX_OUT4
- U19 pad 1: N_1D363273 -> ZT_G1
- U19 pad 10: N_3F511F79 -> ZT_G6
- U19 pad 11: N_3E511DE6 -> FI_OR
- U19 pad 12: N_3D511C53 -> FI_ZN
- U19 pad 13: N_3C511AC0 -> FI_C
- U19 pad 14: A13 -> +5V
- U19 pad 2: N_1E363406 -> ZT_G2
- U19 pad 3: N_1F363599 -> ZT_G5
- U19 pad 4: N_2036372C -> ZT_G3
- U19 pad 5: N_213638BF -> ZT_G4
- U19 pad 6: N_22363A52 -> ZT_G6
- U19 pad 7: OSC_OE -> GND
- U19 pad 8: N_24363D78 -> ZT_G7
- U19 pad 9: N_25363F0B -> ZT_G5
- U2 pad 1: N_01AE718B -> GND
- U2 pad 10: N_609D0961 -> MAR_LOW_IN
- U2 pad 11: DBUS3_2 -> DBUS7
- U2 pad 12: DBUS2_2 -> DBUS6
- U2 pad 13: DBUS1_2 -> DBUS5
- U2 pad 14: DBUS0_2 -> DBUS4
- U2 pad 15: OSC_OE -> GND
- U2 pad 16: A13 -> +5V
- U2 pad 2: N_02AE731E -> GND
- U2 pad 3: ALU_B0_2 -> MARL4
- U2 pad 4: ALU_B1_2 -> MARL5
- U2 pad 5: ALU_B2_2 -> MARL6
- U2 pad 6: ALU_B3_2 -> MARL7
- U2 pad 7: CLK_2 -> CLK
- U2 pad 8: OSC_OE -> GND
- U2 pad 9: N_F9AE64F3 -> MAR_LOW_IN
- U20 pad 1: N_C7D9CE4F -> IROM_OUT
- U20 pad 10: N_1AE011ED -> REG_OUT_N
- U20 pad 11: N_19E0105A -> REG_OUT
- U20 pad 12: N_18E00EC7 -> PC_LOAD_N
- U20 pad 13: N_17E00D34 -> PC_LOAD
- U20 pad 14: A13 -> +5V
- U20 pad 2: N_C8D9CFE2 -> IROM_OUT_N
- U20 pad 3: N_C9D9D175 -> RAM_OUT
- U20 pad 4: N_C2D9C670 -> RAM_OUT_N
- U20 pad 5: N_C3D9C803 -> RAM_IN
- U20 pad 6: N_C4D9C996 -> RAM_IN_N
- U20 pad 7: OSC_OE -> GND
- U20 pad 8: N_CED9D954 -> REG_IN_N
- U20 pad 9: N_CFD9DAE7 -> REG_IN
- U21 pad 1: N_ACB6F990 -> unconnected-(U21-#OE1-Pad1)
- U21 pad 10: N_840AF6E0 -> unconnected-(U21-#E2-Pad10)
- U21 pad 15: OSC_OE -> GND
- U21 pad 16: A13 -> +5V
- U21 pad 2: N_AFB6FE49 -> unconnected-(U21-#OE-Pad2)
- U21 pad 3: N_AEB6FCB6 -> unconnected-(U21-Q0-Pad3)
- U21 pad 4: N_B1B7016F -> unconnected-(U21-Q1-Pad4)
- U21 pad 5: N_B0B6FFDC -> unconnected-(U21-Q2-Pad5)
- U21 pad 6: N_B3B70495 -> unconnected-(U21-Q3-Pad6)
- U21 pad 8: OSC_OE -> GND
- U21 pad 9: N_B4B70628 -> unconnected-(U21-#E1-Pad9)
- U22 pad 1: N_71DB09E5 -> unconnected-(U22-A14-Pad1)
- U22 pad 10: N_10D07A4F -> unconnected-(U22-A0-Pad10)
- U22 pad 11: N_0FD078BC -> unconnected-(U22-I/O0-Pad11)
- U22 pad 12: N_12D07D75 -> unconnected-(U22-I/O1-Pad12)
- U22 pad 13: N_11D07BE2 -> unconnected-(U22-I/O2-Pad13)
- U22 pad 14: OSC_OE -> GND
- U22 pad 15: N_0BD07270 -> unconnected-(U22-I/O3-Pad15)
- U22 pad 16: N_0ED07729 -> unconnected-(U22-I/O4-Pad16)
- U22 pad 17: N_0DD07596 -> unconnected-(U22-I/O5-Pad17)
- U22 pad 18: N_18D086E7 -> unconnected-(U22-I/O6-Pad18)
- U22 pad 19: N_17D08554 -> unconnected-(U22-I/O7-Pad19)
- U22 pad 2: N_6EDB052C -> unconnected-(U22-A12-Pad2)
- U22 pad 20: N_9EC90B14 -> unconnected-(U22-~{CE}-Pad20)
- U22 pad 21: N_9FC90CA7 -> unconnected-(U22-A10-Pad21)
- U22 pad 22: N_A0C90E3A -> unconnected-(U22-~{OE}-Pad22)
- U22 pad 23: N_A1C90FCD -> unconnected-(U22-A11-Pad23)
- U22 pad 24: N_9AC904C8 -> unconnected-(U22-A9-Pad24)
- U22 pad 25: N_9BC9065B -> unconnected-(U22-A8-Pad25)
- U22 pad 26: N_9CC907EE -> unconnected-(U22-A13-Pad26)
- U22 pad 27: N_9DC90981 -> unconnected-(U22-~{WE}-Pad27)
- U22 pad 28: A13 -> +5V
- U22 pad 3: N_6FDB06BF -> unconnected-(U22-A7-Pad3)
- U22 pad 4: N_6CDB0206 -> unconnected-(U22-A6-Pad4)
- U22 pad 5: N_6DDB0399 -> unconnected-(U22-A5-Pad5)
- U22 pad 6: N_6ADAFEE0 -> unconnected-(U22-A4-Pad6)
- U22 pad 7: N_6BDB0073 -> unconnected-(U22-A3-Pad7)
- U22 pad 8: N_78DB14EA -> unconnected-(U22-A2-Pad8)
- U22 pad 9: N_79DB167D -> unconnected-(U22-A1-Pad9)
- U23 pad 14: OSC_OE -> GND
- U23 pad 27: A13 -> +5V
- U23 pad 28: A13 -> +5V
- U24 pad 1: N_1CC9C81B -> unconnected-(U24-A14-Pad1)
- U24 pad 10: N_7CA61BB1 -> unconnected-(U24-A0-Pad10)
- U24 pad 11: N_7BA61A1E -> unconnected-(U24-I/O0-Pad11)
- U24 pad 12: N_7AA6188B -> unconnected-(U24-I/O1-Pad12)
- U24 pad 13: N_79A616F8 -> unconnected-(U24-I/O2-Pad13)
- U24 pad 14: OSC_OE -> GND
- U24 pad 15: N_7FA6206A -> unconnected-(U24-I/O3-Pad15)
- U24 pad 16: N_7EA61ED7 -> unconnected-(U24-I/O4-Pad16)
- U24 pad 17: N_7DA61D44 -> unconnected-(U24-I/O5-Pad17)
- U24 pad 18: N_74A60F19 -> unconnected-(U24-I/O6-Pad18)
- U24 pad 19: N_73A60D86 -> unconnected-(U24-I/O7-Pad19)
- U24 pad 2: N_1DC9C9AE -> unconnected-(U24-A12-Pad2)
- U24 pad 20: N_82A863BA -> unconnected-(U24-~{CE}-Pad20)
- U24 pad 21: N_83A8654D -> unconnected-(U24-A10-Pad21)
- U24 pad 22: N_80A86094 -> unconnected-(U24-~{OE}-Pad22)
- U24 pad 23: N_81A86227 -> unconnected-(U24-A11-Pad23)
- U24 pad 24: N_7EA85D6E -> unconnected-(U24-A9-Pad24)
- U24 pad 25: N_7FA85F01 -> unconnected-(U24-A8-Pad25)
- U24 pad 26: N_7CA85A48 -> unconnected-(U24-A13-Pad26)
- U24 pad 27: N_7DA85BDB -> unconnected-(U24-~{WE}-Pad27)
- U24 pad 28: A13 -> +5V
- U24 pad 3: N_1EC9CB41 -> unconnected-(U24-A7-Pad3)
- U24 pad 4: N_1FC9CCD4 -> unconnected-(U24-A6-Pad4)
- U24 pad 5: N_20C9CE67 -> unconnected-(U24-A5-Pad5)
- U24 pad 6: N_21C9CFFA -> unconnected-(U24-A4-Pad6)
- U24 pad 7: N_22C9D18D -> unconnected-(U24-A3-Pad7)
- U24 pad 8: N_13C9B9F0 -> unconnected-(U24-A2-Pad8)
- U24 pad 9: N_14C9BB83 -> unconnected-(U24-A1-Pad9)
- U25 pad 1: N_8108591C -> RESET_N
- U25 pad 10: N_4C246044 -> +5V
- U25 pad 11: N_4D2461D7 -> unconnected-(U25-QD-Pad11)
- U25 pad 12: N_4E24636A -> STEP2
- U25 pad 13: N_4F2464FD -> STEP1
- U25 pad 14: N_482459F8 -> STEP0
- U25 pad 15: N_49245B8B -> unconnected-(U25-RCO-Pad15)
- U25 pad 16: A13 -> +5V
- U25 pad 2: CLK_2 -> CLK
- U25 pad 3: N_83085C42 -> GND
- U25 pad 4: N_7E085463 -> GND
- U25 pad 5: N_7D0852D0 -> GND
- U25 pad 6: N_80085789 -> GND
- U25 pad 7: N_7F0855F6 -> +5V
- U25 pad 8: OSC_OE -> GND
- U25 pad 9: N_890865B4 -> +5V
- U26 pad 1: N_C67B51D1 -> unconnected-(U26-~{CLR}-Pad1)
- U26 pad 10: N_5521E533 -> unconnected-(U26-ENT-Pad10)
- U26 pad 11: N_5421E3A0 -> unconnected-(U26-QD-Pad11)
- U26 pad 12: N_5721E859 -> unconnected-(U26-QC-Pad12)
- U26 pad 13: N_5621E6C6 -> unconnected-(U26-QB-Pad13)
- U26 pad 14: N_5921EB7F -> unconnected-(U26-QA-Pad14)
- U26 pad 15: N_5821E9EC -> unconnected-(U26-RCO-Pad15)
- U26 pad 16: A13 -> +5V
- U26 pad 3: N_C47B4EAB -> unconnected-(U26-A-Pad3)
- U26 pad 4: N_C97B568A -> unconnected-(U26-B-Pad4)
- U26 pad 5: N_CA7B581D -> unconnected-(U26-C-Pad5)
- U26 pad 6: N_C77B5364 -> unconnected-(U26-D-Pad6)
- U26 pad 7: N_C87B54F7 -> unconnected-(U26-ENP-Pad7)
- U26 pad 8: OSC_OE -> GND
- U26 pad 9: N_BE7B4539 -> unconnected-(U26-~{LOAD}-Pad9)
- U27 pad 1: N_2BF71752 -> unconnected-(U27-~{CLR}-Pad1)
- U27 pad 10: N_97F9CF46 -> unconnected-(U27-ENT-Pad10)
- U27 pad 11: N_98F9D0D9 -> unconnected-(U27-QD-Pad11)
- U27 pad 12: N_95F9CC20 -> unconnected-(U27-QC-Pad12)
- U27 pad 13: N_96F9CDB3 -> unconnected-(U27-QB-Pad13)
- U27 pad 14: N_9BF9D592 -> unconnected-(U27-QA-Pad14)
- U27 pad 15: N_9CF9D725 -> unconnected-(U27-RCO-Pad15)
- U27 pad 16: A13 -> +5V
- U27 pad 3: N_29F7142C -> unconnected-(U27-A-Pad3)
- U27 pad 4: N_28F71299 -> unconnected-(U27-B-Pad4)
- U27 pad 5: N_27F71106 -> unconnected-(U27-C-Pad5)
- U27 pad 6: N_26F70F73 -> unconnected-(U27-D-Pad6)
- U27 pad 7: N_25F70DE0 -> unconnected-(U27-ENP-Pad7)
- U27 pad 8: OSC_OE -> GND
- U27 pad 9: N_33F723EA -> unconnected-(U27-~{LOAD}-Pad9)
- U28 pad 1: N_3EE78FB7 -> unconnected-(U28-~{CLR}-Pad1)
- U28 pad 10: N_8D86F185 -> unconnected-(U28-ENT-Pad10)
- U28 pad 11: N_8C86EFF2 -> unconnected-(U28-QD-Pad11)
- U28 pad 12: N_8B86EE5F -> unconnected-(U28-QC-Pad12)
- U28 pad 13: N_8A86ECCC -> unconnected-(U28-QB-Pad13)
- U28 pad 14: N_8986EB39 -> unconnected-(U28-QA-Pad14)
- U28 pad 15: N_8886E9A6 -> unconnected-(U28-RCO-Pad15)
- U28 pad 16: A13 -> +5V
- U28 pad 3: N_40E792DD -> unconnected-(U28-A-Pad3)
- U28 pad 4: N_39E787D8 -> unconnected-(U28-B-Pad4)
- U28 pad 5: N_3AE7896B -> unconnected-(U28-C-Pad5)
- U28 pad 6: N_3BE78AFE -> unconnected-(U28-D-Pad6)
- U28 pad 7: N_3CE78C91 -> unconnected-(U28-ENP-Pad7)
- U28 pad 8: OSC_OE -> GND
- U28 pad 9: N_36E7831F -> unconnected-(U28-~{LOAD}-Pad9)
- U29 pad 1: N_A4635538 -> unconnected-(U29-~{CLR}-Pad1)
- U29 pad 10: N_D05EDB98 -> unconnected-(U29-ENT-Pad10)
- U29 pad 11: N_D15EDD2B -> unconnected-(U29-QD-Pad11)
- U29 pad 12: N_D25EDEBE -> unconnected-(U29-QC-Pad12)
- U29 pad 13: N_D35EE051 -> unconnected-(U29-QB-Pad13)
- U29 pad 14: N_D45EE1E4 -> unconnected-(U29-QA-Pad14)
- U29 pad 15: N_D55EE377 -> unconnected-(U29-RCO-Pad15)
- U29 pad 16: A13 -> +5V
- U29 pad 3: N_A663585E -> unconnected-(U29-A-Pad3)
- U29 pad 4: N_A9635D17 -> unconnected-(U29-B-Pad4)
- U29 pad 5: N_A8635B84 -> unconnected-(U29-C-Pad5)
- U29 pad 6: N_AB63603D -> unconnected-(U29-D-Pad6)
- U29 pad 7: N_AA635EAA -> unconnected-(U29-ENP-Pad7)
- U29 pad 8: OSC_OE -> GND
- U29 pad 9: N_9C6348A0 -> unconnected-(U29-~{LOAD}-Pad9)
- U3 pad 1: N_668AD34C -> GND
- U3 pad 10: N_E88AEC34 -> MAR_HIGH_IN
- U3 pad 11: DBUS3_2 -> DBUS3
- U3 pad 12: DBUS2_2 -> DBUS2
- U3 pad 13: DBUS1_2 -> DBUS1
- U3 pad 14: DBUS0_2 -> DBUS0
- U3 pad 15: OSC_OE -> GND
- U3 pad 16: A13 -> +5V
- U3 pad 2: N_698AD805 -> GND
- U3 pad 3: ALU_A4_2 -> MARH0
- U3 pad 4: ALU_A5_2 -> MARH1
- U3 pad 5: ALU_A6_2 -> MARH2
- U3 pad 6: ALU_A7_2 -> MARH3
- U3 pad 7: CLK_2 -> CLK
- U3 pad 8: OSC_OE -> GND
- U3 pad 9: N_6E8ADFE4 -> MAR_HIGH_IN
- U30 pad 1: N_F9082CAA -> unconnected-(U30-~{CLR}-Pad1)
- U30 pad 10: N_A1DE366E -> unconnected-(U30-ENT-Pad10)
- U30 pad 11: N_A2DE3801 -> unconnected-(U30-QD-Pad11)
- U30 pad 12: N_9FDE3348 -> unconnected-(U30-QC-Pad12)
- U30 pad 13: N_A0DE34DB -> unconnected-(U30-QB-Pad13)
- U30 pad 14: N_A5DE3CBA -> unconnected-(U30-QA-Pad14)
- U30 pad 15: N_A6DE3E4D -> unconnected-(U30-RCO-Pad15)
- U30 pad 16: A13 -> +5V
- U30 pad 3: N_F7082984 -> unconnected-(U30-A-Pad3)
- U30 pad 4: N_F60827F1 -> unconnected-(U30-B-Pad4)
- U30 pad 5: N_F508265E -> unconnected-(U30-C-Pad5)
- U30 pad 6: N_F40824CB -> unconnected-(U30-D-Pad6)
- U30 pad 7: N_F3082338 -> unconnected-(U30-ENP-Pad7)
- U30 pad 8: OSC_OE -> GND
- U30 pad 9: N_F1082012 -> unconnected-(U30-~{LOAD}-Pad9)
- U31 pad 1: N_F4CA32C9 -> unconnected-(U31-NC-Pad1)
- U31 pad 14: OSC_OE -> GND
- U31 pad 26: N_C746A5D2 -> unconnected-(U31-NC-Pad26)
- U31 pad 28: A13 -> +5V
- U32 pad 1: OSC_OE -> GND
- U32 pad 10: ALU_LOAD_LOW -> A_IN
- U32 pad 15: OSC_OE -> GND
- U32 pad 16: A13 -> +5V
- U32 pad 2: OSC_OE -> GND
- U32 pad 8: OSC_OE -> GND
- U32 pad 9: ALU_LOAD_LOW -> A_IN
- U33 pad 1: OSC_OE -> GND
- U33 pad 10: ALU_LOAD_LOW -> TEMP_IN
- U33 pad 15: OSC_OE -> GND
- U33 pad 16: A13 -> +5V
- U33 pad 2: OSC_OE -> GND
- U33 pad 3: ALU_B0 -> ALU_B_RAW0
- U33 pad 4: ALU_B1 -> ALU_B_RAW1
- U33 pad 5: ALU_B2 -> ALU_B_RAW2
- U33 pad 6: ALU_B3 -> ALU_B_RAW3
- U33 pad 8: OSC_OE -> GND
- U33 pad 9: ALU_LOAD_LOW -> TEMP_IN
- U34 pad 1: OSC_OE -> GND
- U34 pad 10: ALU_LOAD_HIGH -> A_IN
- U34 pad 11: DBUS3 -> DBUS7
- U34 pad 12: DBUS2 -> DBUS6
- U34 pad 13: DBUS1 -> DBUS5
- U34 pad 14: DBUS0 -> DBUS4
- U34 pad 15: OSC_OE -> GND
- U34 pad 16: A13 -> +5V
- U34 pad 2: OSC_OE -> GND
- U34 pad 8: OSC_OE -> GND
- U34 pad 9: ALU_LOAD_HIGH -> A_IN
- U35 pad 1: OSC_OE -> GND
- U35 pad 10: ALU_LOAD_HIGH -> TEMP_IN
- U35 pad 11: DBUS3 -> DBUS7
- U35 pad 12: DBUS2 -> DBUS6
- U35 pad 13: DBUS1 -> DBUS5
- U35 pad 14: DBUS0 -> DBUS4
- U35 pad 15: OSC_OE -> GND
- U35 pad 16: A13 -> +5V
- U35 pad 2: OSC_OE -> GND
- U35 pad 3: ALU_B4 -> ALU_B_RAW4
- U35 pad 4: ALU_B5 -> ALU_B_RAW5
- U35 pad 5: ALU_B6 -> ALU_B_RAW6
- U35 pad 6: ALU_B7 -> ALU_B_RAW7
- U35 pad 8: OSC_OE -> GND
- U35 pad 9: ALU_LOAD_HIGH -> TEMP_IN
- U36 pad 16: A13 -> +5V
- U36 pad 7: OSC_OE -> SU
- U36 pad 8: OSC_OE -> GND
- U37 pad 16: A13 -> +5V
- U37 pad 8: OSC_OE -> GND
- U37 pad 9: N_8E280B8F -> C_COMPUTED
- U38 pad 1: OSC_OE -> GND
- U38 pad 10: N_C8E3F736 -> ALU_S1
- U38 pad 11: N_C9E3F8C9 -> ALU_AND1
- U38 pad 12: N_C6E3F410 -> ALU_OR1
- U38 pad 13: N_C7E3F5A3 -> ALU_B1
- U38 pad 14: N_CCE3FD82 -> ALU_SEL0
- U38 pad 15: OSC_OE -> GND
- U38 pad 16: A13 -> +5V
- U38 pad 2: N_019903EF -> ALU_SEL1
- U38 pad 3: ALU_S3 -> ALU_B0
- U38 pad 4: ALU_S2 -> ALU_OR0
- U38 pad 5: ALU_S1 -> ALU_AND0
- U38 pad 8: OSC_OE -> GND
- U39 pad 1: OSC_OE -> GND
- U39 pad 10: N_3FB8DFE3 -> ALU_S3
- U39 pad 11: N_3EB8DE50 -> ALU_AND3
- U39 pad 12: N_41B8E309 -> ALU_OR3
- U39 pad 13: N_40B8E176 -> ALU_B3
- U39 pad 14: N_43B8E62F -> ALU_SEL0
- U39 pad 15: OSC_OE -> GND
- U39 pad 16: A13 -> +5V
- U39 pad 2: N_1ABBD588 -> ALU_SEL1
- U39 pad 3: ALU_S7 -> ALU_B2
- U39 pad 4: ALU_S6 -> ALU_OR2
- U39 pad 5: ALU_S5 -> ALU_AND2
- U39 pad 6: ALU_S4 -> ALU_S2
- U39 pad 8: OSC_OE -> GND
- U4 pad 1: N_57FCE7D5 -> GND
- U4 pad 10: N_68210D7F -> FI_LATCH_N
- U4 pad 11: DBUS3_2 -> GND
- U4 pad 12: DBUS2_2 -> GND
- U4 pad 13: DBUS1_2 -> C_COMPUTED
- U4 pad 14: DBUS0_2 -> Z_COMPUTED
- U4 pad 15: OSC_OE -> GND
- U4 pad 16: A13 -> +5V
- U4 pad 2: N_54FCE31C -> GND
- U4 pad 3: ALU_B4_2 -> Z
- U4 pad 4: ALU_B5_2 -> C
- U4 pad 5: ALU_B6_2 -> unconnected-(U4-Q2-Pad5)
- U4 pad 6: ALU_B7_2 -> unconnected-(U4-Q3-Pad6)
- U4 pad 7: CLK_2 -> CLK
- U4 pad 8: OSC_OE -> GND
- U4 pad 9: N_5FFCF46D -> FI_LATCH_N
- U40 pad 1: OSC_OE -> GND
- U40 pad 10: N_B7A39887 -> ALU_S5
- U40 pad 11: N_B6A396F4 -> ALU_AND5
- U40 pad 12: N_B9A39BAD -> ALU_OR5
- U40 pad 13: N_B8A39A1A -> ALU_B5
- U40 pad 14: N_B3A3923B -> ALU_SEL0
- U40 pad 15: OSC_OE -> GND
- U40 pad 16: A13 -> +5V
- U40 pad 2: N_86D530D4 -> ALU_SEL1
- U40 pad 3: N_87D53267 -> ALU_B4
- U40 pad 4: N_84D52DAE -> ALU_OR4
- U40 pad 5: N_85D52F41 -> ALU_AND4
- U40 pad 6: N_82D52A88 -> ALU_S4
- U40 pad 8: OSC_OE -> GND
- U41 pad 1: OSC_OE -> GND
- U41 pad 10: N_FA7B829A -> ALU_S7
- U41 pad 11: N_FB7B842D -> ALU_AND7
- U41 pad 12: N_F87B7F74 -> ALU_OR7
- U41 pad 13: N_F97B8107 -> ALU_B7
- U41 pad 14: N_F67B7C4E -> ALU_SEL0
- U41 pad 15: OSC_OE -> GND
- U41 pad 16: A13 -> +5V
- U41 pad 2: N_EE50F97B -> ALU_SEL1
- U41 pad 3: N_ED50F7E8 -> ALU_B6
- U41 pad 4: N_F45102ED -> ALU_OR6
- U41 pad 5: N_F351015A -> ALU_AND6
- U41 pad 6: N_F250FFC7 -> ALU_S6
- U41 pad 8: OSC_OE -> GND
- U42 pad 1: VCC -> GND
- U42 pad 10: OSC_OE -> GND
- U42 pad 19: N_C627A7AA -> EO_N
- U42 pad 20: A13 -> +5V
- U43 pad 1: N_C4617358 -> GND
- U43 pad 10: N_8D68ACB8 -> unconnected-(U43-~{2Y2}-Pad10)
- U43 pad 11: N_8E68AE4B -> unconnected-(U43-~{2Y1}-Pad11)
- U43 pad 12: N_8F68AFDE -> unconnected-(U43-~{2Y0}-Pad12)
- U43 pad 13: N_9068B171 -> unconnected-(U43-2A1-Pad13)
- U43 pad 14: N_9168B304 -> unconnected-(U43-2A0-Pad14)
- U43 pad 15: N_9268B497 -> unconnected-(U43-~{2E}-Pad15)
- U43 pad 16: A13 -> +5V
- U43 pad 4: N_C9617B37 -> REGSEL_Y0
- U43 pad 5: N_C86179A4 -> REGSEL_Y1
- U43 pad 6: N_CB617E5D -> REGSEL_Y2
- U43 pad 7: N_CA617CCA -> REGSEL_Y3
- U43 pad 8: OSC_OE -> GND
- U43 pad 9: N_BC6166C0 -> unconnected-(U43-~{2Y3}-Pad9)
- U44 pad 1: N_3E2662B9 -> REGSEL_Y0
- U44 pad 10: N_5F6D1DAB -> REG_IN_N
- U44 pad 15: OSC_OE -> GND
- U44 pad 16: A13 -> +5V
- U44 pad 2: N_3B265E00 -> REG_OUT_N
- U44 pad 3: N_3C265F93 -> DBUS0
- U44 pad 4: N_41266772 -> DBUS1
- U44 pad 5: N_42266905 -> DBUS2
- U44 pad 6: N_3F26644C -> DBUS3
- U44 pad 8: OSC_OE -> GND
- U44 pad 9: N_46266F51 -> REGSEL_Y0
- U45 pad 1: N_4303C05A -> REGSEL_Y0
- U45 pad 10: N_E8E7E6DE -> REG_IN_N
- U45 pad 11: DBUS3 -> DBUS7
- U45 pad 12: DBUS2 -> DBUS6
- U45 pad 13: DBUS1 -> DBUS5
- U45 pad 14: DBUS0 -> DBUS4
- U45 pad 15: OSC_OE -> GND
- U45 pad 16: A13 -> +5V
- U45 pad 2: N_4203BEC7 -> REG_OUT_N
- U45 pad 3: N_4103BD34 -> DBUS4
- U45 pad 4: N_4003BBA1 -> DBUS5
- U45 pad 5: N_3F03BA0E -> DBUS6
- U45 pad 6: N_3E03B87B -> DBUS7
- U45 pad 8: OSC_OE -> GND
- U45 pad 9: N_3B03B3C2 -> REGSEL_Y0
- U46 pad 1: N_9474D903 -> REGSEL_Y1
- U46 pad 10: N_E6F1EB49 -> REG_IN_N
- U46 pad 15: OSC_OE -> GND
- U46 pad 16: A13 -> +5V
- U46 pad 2: N_9574DA96 -> REG_OUT_N
- U46 pad 3: N_9674DC29 -> DBUS0
- U46 pad 4: N_9774DDBC -> DBUS1
- U46 pad 5: N_9874DF4F -> DBUS2
- U46 pad 6: N_9974E0E2 -> DBUS3
- U46 pad 8: OSC_OE -> GND
- U46 pad 9: N_9C74E59B -> REGSEL_Y1
- U47 pad 1: N_990284C4 -> REGSEL_Y1
- U47 pad 10: N_D2F74C1C -> REG_IN_N
- U47 pad 11: DBUS3 -> DBUS7
- U47 pad 12: DBUS2 -> DBUS6
- U47 pad 13: DBUS1 -> DBUS5
- U47 pad 14: DBUS0 -> DBUS4
- U47 pad 15: OSC_OE -> GND
- U47 pad 16: A13 -> +5V
- U47 pad 2: N_9C02897D -> REG_OUT_N
- U47 pad 3: N_9B0287EA -> DBUS4
- U47 pad 4: N_9602800B -> DBUS5
- U47 pad 5: N_95027E78 -> DBUS6
- U47 pad 6: N_98028331 -> DBUS7
- U47 pad 8: OSC_OE -> GND
- U47 pad 9: N_9102782C -> REGSEL_Y1
- U48 pad 1: N_93165C85 -> REGSEL_Y2
- U48 pad 10: N_4133F0EF -> REG_IN_N
- U48 pad 15: OSC_OE -> GND
- U48 pad 16: A13 -> +5V
- U48 pad 2: N_901657CC -> REG_OUT_N
- U48 pad 3: N_9116595F -> DBUS0
- U48 pad 4: N_8E1654A6 -> DBUS1
- U48 pad 5: N_8F165639 -> DBUS2
- U48 pad 6: N_8C165180 -> DBUS3
- U48 pad 8: OSC_OE -> GND
- U48 pad 9: N_9B16691D -> REGSEL_Y2
- U49 pad 1: N_F754ED86 -> REGSEL_Y2
- U49 pad 10: N_10B23582 -> REG_IN_N
- U49 pad 11: DBUS3 -> DBUS7
- U49 pad 12: DBUS2 -> DBUS6
- U49 pad 13: DBUS1 -> DBUS5
- U49 pad 14: DBUS0 -> DBUS4
- U49 pad 15: OSC_OE -> GND
- U49 pad 16: A13 -> +5V
- U49 pad 2: N_F654EBF3 -> REG_OUT_N
- U49 pad 3: N_F554EA60 -> DBUS4
- U49 pad 4: N_FC54F565 -> DBUS5
- U49 pad 5: N_FB54F3D2 -> DBUS6
- U49 pad 6: N_FA54F23F -> DBUS7
- U49 pad 8: OSC_OE -> GND
- U49 pad 9: N_FF54FA1E -> REGSEL_Y2
- U5 pad 1: N_BCD94996 -> unconnected-(U5-S1-Pad1)
- U5 pad 10: N_F00EF052 -> unconnected-(U5-S3-Pad10)
- U5 pad 13: N_EF0EEEBF -> unconnected-(U5-S2-Pad13)
- U5 pad 16: A13 -> +5V
- U5 pad 4: N_C1D95175 -> unconnected-(U5-S0-Pad4)
- U5 pad 7: N_BED94CBC -> unconnected-(U5-CIN-Pad7)
- U5 pad 8: OSC_OE -> GND
- U50 pad 1: N_9B036188 -> REGSEL_Y3
- U50 pad 10: N_BE52D4A8 -> REG_IN_N
- U50 pad 15: OSC_OE -> GND
- U50 pad 16: A13 -> +5V
- U50 pad 2: N_9E036641 -> REG_OUT_N
- U50 pad 3: N_9D0364AE -> DBUS0
- U50 pad 4: N_A0036967 -> DBUS1
- U50 pad 5: N_9F0367D4 -> DBUS2
- U50 pad 6: N_A2036C8D -> DBUS3
- U50 pad 8: OSC_OE -> GND
- U50 pad 9: N_930354F0 -> REGSEL_Y3
- U51 pad 1: N_3626FFC7 -> REGSEL_Y3
- U51 pad 10: N_3664F1D5 -> REG_IN_N
- U51 pad 11: DBUS3 -> DBUS7
- U51 pad 12: DBUS2 -> DBUS6
- U51 pad 13: DBUS1 -> DBUS5
- U51 pad 14: DBUS0 -> DBUS4
- U51 pad 15: OSC_OE -> GND
- U51 pad 16: A13 -> +5V
- U51 pad 2: N_3727015A -> REG_OUT_N
- U51 pad 3: N_382702ED -> DBUS4
- U51 pad 4: N_3126F7E8 -> DBUS5
- U51 pad 5: N_3226F97B -> DBUS6
- U51 pad 6: N_3326FB0E -> DBUS7
- U51 pad 8: OSC_OE -> GND
- U51 pad 9: N_2E26F32F -> REGSEL_Y3
- U52 pad 10: OSC_OE -> PC_INC
- U52 pad 16: A13 -> +5V
- U52 pad 3: N_43F21C98 -> MARL0
- U52 pad 4: N_4AF2279D -> MARL1
- U52 pad 5: N_49F2260A -> MARL2
- U52 pad 6: N_48F22477 -> MARL3
- U52 pad 7: OSC_OE -> PC_INC
- U52 pad 8: OSC_OE -> GND
- U52 pad 9: N_3DF21326 -> PC_LOAD_N
- U53 pad 16: A13 -> +5V
- U53 pad 3: N_DF15BAD7 -> MARL4
- U53 pad 4: N_DC15B61E -> MARL5
- U53 pad 5: N_DD15B7B1 -> MARL6
- U53 pad 6: N_DA15B2F8 -> MARL7
- U53 pad 8: OSC_OE -> GND
- U53 pad 9: N_D915B165 -> PC_LOAD_N
- U54 pad 11: N_84E0AC1F -> unconnected-(U54-QD-Pad11)
- U54 pad 12: N_85E0ADB2 -> unconnected-(U54-QC-Pad12)
- U54 pad 15: N_80E0A5D3 -> unconnected-(U54-RCO-Pad15)
- U54 pad 16: A13 -> +5V
- U54 pad 3: N_71A4761A -> MARH0
- U54 pad 4: N_6CA46E3B -> MARH1
- U54 pad 5: N_6BA46CA8 -> MARH2
- U54 pad 6: N_6EA47161 -> MARH3
- U54 pad 8: OSC_OE -> GND
- U54 pad 9: N_67A4665C -> PC_LOAD_N
- U55 pad 1: N_6B16C733 -> unconnected-(U55-#OE1-Pad1)
- U55 pad 10: N_97DB49B9 -> IR_IN
- U55 pad 15: OSC_OE -> GND
- U55 pad 16: A13 -> +5V
- U55 pad 2: N_6C16C8C6 -> unconnected-(U55-#OE-Pad2)
- U55 pad 3: REG_SEL0 -> IR_RS0
- U55 pad 4: REG_SEL1 -> IR_RS1
- U55 pad 5: N_6F16CD7F -> IR_RD0
- U55 pad 6: N_7016CF12 -> IR_RD1
- U55 pad 8: OSC_OE -> GND
- U55 pad 9: N_7316D3CB -> IR_IN
- U56 pad 1: N_1A437F4A -> unconnected-(U56-#OE1-Pad1)
- U56 pad 10: N_D241AD0E -> IR_IN
- U56 pad 11: DBUS3 -> DBUS7
- U56 pad 12: DBUS2 -> DBUS6
- U56 pad 13: DBUS1 -> DBUS5
- U56 pad 14: DBUS0 -> DBUS4
- U56 pad 15: OSC_OE -> GND
- U56 pad 16: A13 -> +5V
- U56 pad 2: N_19437DB7 -> unconnected-(U56-#OE-Pad2)
- U56 pad 3: N_18437C24 -> OPCODE0
- U56 pad 4: N_17437A91 -> OPCODE1
- U56 pad 5: N_164378FE -> OPCODE2
- U56 pad 6: N_1543776B -> OPCODE3
- U56 pad 8: OSC_OE -> GND
- U56 pad 9: N_124372B2 -> IR_IN
- U57 pad 1: N_14C850E9 -> GND
- U57 pad 10: N_9057459B -> C
- U57 pad 11: N_8F574408 -> IROM_OUT
- U57 pad 12: N_925748C1 -> RAM_OUT
- U57 pad 13: N_9157472E -> RAM_IN
- U57 pad 14: OSC_OE -> GND
- U57 pad 15: N_93574A54 -> IR_IN
- U57 pad 16: N_96574F0D -> MAR_LOW_IN
- U57 pad 17: N_95574D7A -> MAR_HIGH_IN
- U57 pad 18: N_88573903 -> PC_INC
- U57 pad 19: N_87573770 -> PC_LOAD
- U57 pad 2: N_11C84C30 -> GND
- U57 pad 20: OSC_OE -> GND
- U57 pad 21: N_FF4FA593 -> GND
- U57 pad 22: OSC_OE -> GND
- U57 pad 23: N_014FA8B9 -> GND
- U57 pad 24: N_024FAA4C -> GND
- U57 pad 25: N_034FABDF -> OPCODE3
- U57 pad 26: N_044FAD72 -> GND
- U57 pad 27: N_054FAF05 -> +5V
- U57 pad 28: A13 -> +5V
- U57 pad 3: N_12C84DC3 -> OPCODE2
- U57 pad 4: N_17C855A2 -> OPCODE1
- U57 pad 5: N_18C85735 -> OPCODE0
- U57 pad 6: N_15C8527C -> STEP2
- U57 pad 7: N_16C8540F -> STEP1
- U57 pad 8: N_1BC85BEE -> STEP0
- U57 pad 9: N_1CC85D81 -> Z
- U58 pad 1: N_23F5A020 -> GND
- U58 pad 10: N_ABAAF930 -> C
- U58 pad 11: N_ACAAFAC3 -> RS_SEL
- U58 pad 12: N_ADAAFC56 -> REG_IN
- U58 pad 13: N_AEAAFDE9 -> REG_OUT
- U58 pad 14: OSC_OE -> GND
- U58 pad 15: N_B0AB010F -> A_IN
- U58 pad 16: N_B1AB02A2 -> TEMP_IN
- U58 pad 17: N_B2AB0435 -> ALU_SEL0
- U58 pad 18: N_B3AB05C8 -> ALU_SEL1
- U58 pad 19: N_B4AB075B -> SU
- U58 pad 2: N_26F5A4D9 -> GND
- U58 pad 20: OSC_OE -> GND
- U58 pad 21: N_3CB29938 -> GND
- U58 pad 22: OSC_OE -> GND
- U58 pad 23: N_3EB29C5E -> GND
- U58 pad 24: N_41B2A117 -> GND
- U58 pad 25: N_40B29F84 -> OPCODE3
- U58 pad 26: N_43B2A43D -> GND
- U58 pad 27: N_42B2A2AA -> +5V
- U58 pad 28: A13 -> +5V
- U58 pad 3: N_25F5A346 -> OPCODE2
- U58 pad 4: N_28F5A7FF -> OPCODE1
- U58 pad 5: N_27F5A66C -> OPCODE0
- U58 pad 6: N_2AF5AB25 -> STEP2
- U58 pad 7: N_29F5A992 -> STEP1
- U58 pad 8: N_2CF5AE4B -> STEP0
- U58 pad 9: N_2BF5ACB8 -> Z
- U59 pad 1: A14 -> GND
- U59 pad 10: A0 -> C
- U59 pad 11: D0 -> EO
- U59 pad 12: D1 -> FI_ZN
- U59 pad 13: D2 -> FI_C
- U59 pad 14: OSC_OE -> GND
- U59 pad 15: D3 -> HLT
- U59 pad 2: A12 -> GND
- U59 pad 20: OSC_OE -> GND
- U59 pad 21: A10 -> GND
- U59 pad 22: OSC_OE -> GND
- U59 pad 23: A11 -> GND
- U59 pad 24: A9 -> GND
- U59 pad 25: A8 -> OPCODE3
- U59 pad 26: N_E42EFFCC -> GND
- U59 pad 27: A13 -> +5V
- U59 pad 28: A13 -> +5V
- U59 pad 3: A7 -> OPCODE2
- U59 pad 4: A6 -> OPCODE1
- U59 pad 5: A5 -> OPCODE0
- U59 pad 6: A4 -> STEP2
- U59 pad 7: A3 -> STEP1
- U59 pad 8: A2 -> STEP0
- U59 pad 9: A1 -> Z
- U6 pad 1: N_2D5D11FF -> unconnected-(U6-S1-Pad1)
- U6 pad 10: N_388308DD -> unconnected-(U6-S3-Pad10)
- U6 pad 13: N_35830424 -> unconnected-(U6-S2-Pad13)
- U6 pad 16: A13 -> +5V
- U6 pad 4: N_285D0A20 -> unconnected-(U6-S0-Pad4)
- U6 pad 8: OSC_OE -> GND
- U6 pad 9: N_355D1E97 -> unconnected-(U6-COUT-Pad9)
- U60 pad 1: N_1BA0C04B -> unconnected-(U60-NC-Pad1)
- U60 pad 14: OSC_OE -> GND
- U60 pad 20: OSC_OE -> GND
- U60 pad 22: OSC_OE -> IROM_OUT_N
- U60 pad 26: N_F9114038 -> unconnected-(U60-NC-Pad26)
- U60 pad 27: A13 -> +5V
- U60 pad 28: A13 -> +5V
- U61 pad 1: A7 -> MARL7
- U61 pad 12: OSC_OE -> GND
- U61 pad 18: RAM_CS -> GND
- U61 pad 19: A10 -> MARH2
- U61 pad 2: A6 -> MARL6
- U61 pad 20: RAM_OE -> RAM_OUT_N
- U61 pad 21: RAM_WE -> RAM_IN_N
- U61 pad 22: A9 -> MARH1
- U61 pad 23: A8 -> MARH0
- U61 pad 24: A13 -> +5V
- U61 pad 3: A5 -> MARL5
- U61 pad 4: A4 -> MARL4
- U61 pad 5: A3 -> MARL3
- U61 pad 6: A2 -> MARL2
- U61 pad 7: A1 -> MARL1
- U61 pad 8: A0 -> MARL0
- U62 pad 1: A13 -> +5V
- U62 pad 2: OSC_OE -> GND
- U62 pad 4: A13 -> +5V
- U63 pad 10: N_CE0F87F6 -> unconnected-(U63-5Y-Pad10)
- U63 pad 11: N_CF0F8989 -> unconnected-(U63-5A-Pad11)
- U63 pad 12: N_CC0F84D0 -> unconnected-(U63-6Y-Pad12)
- U63 pad 13: N_CD0F8663 -> unconnected-(U63-6A-Pad13)
- U63 pad 14: A13 -> +5V
- U63 pad 3: N_A96CA69C -> unconnected-(U63-2A-Pad3)
- U63 pad 4: N_A86CA509 -> unconnected-(U63-2Y-Pad4)
- U63 pad 5: N_A76CA376 -> unconnected-(U63-3A-Pad5)
- U63 pad 6: N_A66CA1E3 -> unconnected-(U63-3Y-Pad6)
- U63 pad 7: OSC_OE -> GND
- U63 pad 8: N_B46CB7ED -> unconnected-(U63-4Y-Pad8)
- U63 pad 9: N_B36CB65A -> unconnected-(U63-4A-Pad9)
- U7 pad 1: N_12D80E00 -> ALU_B_RAW0
- U7 pad 10: N_DA1E5590 -> SU
- U7 pad 11: N_DB1E5723 -> ALU_B3
- U7 pad 12: N_DC1E58B6 -> ALU_B_RAW3
- U7 pad 13: N_DD1E5A49 -> SU
- U7 pad 14: A13 -> +5V
- U7 pad 2: N_15D812B9 -> SU
- U7 pad 3: N_14D81126 -> ALU_B0
- U7 pad 4: N_17D815DF -> ALU_B_RAW1
- U7 pad 5: N_16D8144C -> SU
- U7 pad 6: N_19D81905 -> ALU_B1
- U7 pad 7: OSC_OE -> GND
- U7 pad 8: N_1BD81C2B -> ALU_B2
- U7 pad 9: N_1AD81A98 -> ALU_B_RAW2
- U8 pad 1: N_83AB8849 -> ALU_B_RAW4
- U8 pad 10: N_C007D67B -> SU
- U8 pad 11: N_BF07D4E8 -> ALU_B7
- U8 pad 12: N_C207D9A1 -> ALU_B_RAW7
- U8 pad 13: N_C107D80E -> SU
- U8 pad 14: A13 -> +5V
- U8 pad 2: N_80AB8390 -> SU
- U8 pad 3: N_81AB8523 -> ALU_B4
- U8 pad 4: N_86AB8D02 -> ALU_B_RAW5
- U8 pad 5: N_87AB8E95 -> SU
- U8 pad 6: N_84AB89DC -> ALU_B5
- U8 pad 7: OSC_OE -> GND
- U8 pad 8: N_8AAB934E -> ALU_B6
- U8 pad 9: N_8BAB94E1 -> ALU_B_RAW6
- U9 pad 1: N_87E9822A -> GND
- U9 pad 10: N_0E97CEEE -> IR_RD1
- U9 pad 11: N_0F97D081 -> IR_RS1
- U9 pad 12: N_0C97CBC8 -> unconnected-(U9-2I2-Pad12)
- U9 pad 13: N_0D97CD5B -> unconnected-(U9-2I3-Pad13)
- U9 pad 14: N_1297D53A -> RS_SEL
- U9 pad 15: N_1397D6CD -> GND
- U9 pad 16: A13 -> +5V
- U9 pad 2: N_86E98097 -> GND
- U9 pad 3: N_85E97F04 -> unconnected-(U9-1I3-Pad3)
- U9 pad 4: N_84E97D71 -> unconnected-(U9-1I2-Pad4)
- U9 pad 5: N_83E97BDE -> IR_RS0
- U9 pad 6: N_82E97A4B -> IR_RD0
- U9 pad 7: N_81E978B8 -> REG_SEL0
- U9 pad 8: OSC_OE -> GND
- U9 pad 9: N_7FE97592 -> REG_SEL1
Routing:
- net GND: track 0.00 -> 1275.6 mm, vias 0 -> 36
- net +5V: track 0.00 -> 1026.4 mm, vias 0 -> 47
- net CLK: track 0.00 -> 438.9 mm, vias 0 -> 24
- net DBUS6: track 0.00 -> 412.6 mm, vias 0 -> 10
- net DBUS7: track 0.00 -> 408.5 mm, vias 0 -> 10
- net DBUS4: track 0.00 -> 395.0 mm, vias 0 -> 15
- net DBUS0: track 0.00 -> 390.5 mm, vias 0 -> 14
- net DBUS5: track 0.00 -> 378.5 mm, vias 0 -> 11
- net DBUS1: track 0.00 -> 375.2 mm, vias 0 -> 12
- net DBUS3: track 0.00 -> 359.0 mm, vias 0 -> 12
- net DBUS2: track 0.00 -> 353.3 mm, vias 0 -> 12
- net REG_OUT_N: track 0.00 -> 319.3 mm, vias 0 -> 12
- net REG_IN_N: track 0.00 -> 293.9 mm, vias 0 -> 11
- net ALU_B6: track 0.00 -> 228.0 mm, vias 0 -> 6
- net RESET_N: track 0.00 -> 203.5 mm, vias 0 -> 6
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