File: 8-Bit-CPU-main/kicad_files/8-bit cpu.kicad_sch (KiCad schematic)
At the start: 97 parts, among them SW1 HX 3X4X2-2P-1.6N TACTILE SWIT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, U1 74HC173D,653, U10 74HC153D,653, U11 74HC153D,653, U12 74HC153D,653, U13 74HC245D,653, U14 74HC08D,653, U15 74HC08D,653, U16 74HC32D,653, U17 74HC32D,653, U18 74HC32D,653, U19 74HC32D,653, U2 74HC173D,653, U20 74HC04D,653, U21 74HC173D,653, U22 AT28C256-15SU, U23 AT28C256-15SU, U24 AT28C256-15SU, U25 SN74HC161DR, U26 SN74HC161DR, U27 SN74HC161DR, U28 SN74HC161DR, U29 SN74HC161DR, U3 74HC173D,653, U30 SN74HC161DR, U31 AT28C64B-15PU, U32 74HC173D,653, U33 74HC173D,653, U34 74HC173D,653, U35 74HC173D,653, U36 CD74HC283M96, U37 CD74HC283M96, U38 74HC153D,653, U39 74HC153D,653, U4 74HC173D,653, U40 74HC153D,653, U41 74HC153D,653, U42 74HC245D,653, U43 74HC139D,653, U44 74HC173D,653, U45 74HC173D,653, U46 74HC173D,653, U47 74HC173D,653, U48 74HC173D,653, U49 74HC173D,653, U5 CD74HC283M96, U50 74HC173D,653, U51 74HC173D,653, U52 SN74HC161DR, U53 SN74HC161DR, U54 SN74HC161DR, U55 74HC173D,653, U56 74HC173D,653, U57 AT28C256-15SU, U58 AT28C256-15SU, U59 AT28C256-15SU, U6 CD74HC283M96, U60 AT28C64B-15PU, U61 HM6116LP-4, U62 OT70501MJBA4SL, U63 SN74HC14DR, U7 SN74HC86DR, U8 SN74HC86DR, U9 74HC153D,653

Commit message: Add files via upload
Parts:
- U13, U21, U22, U23, U24, U26, U27, U28, U29, U30, U31, U5, U6: now not fitted
Connections:
- net RAM_CS is gone; now on net GND: U61.18 (CS)
- net RAM_OE is gone; now on net RAM_OUT_N: U61.20 (OE)
- net RAM_WE is gone; now on net RAM_IN_N: U61.21 (WE)
- net VCC is gone; now on net GND: U42.1 (DIR)
- net +5V: now also C1.1, C10.1, C11.1, C12.1, C13.1, C14.1, C15.1, C16.1, C17.1, C18.1, C19.1, C2.1, C20.1, C21.1, C22.1, C23.1, C24.1, C25.1, C26.1, C27.1, C28.1, C29.1, C3.1, C30.1, C4.1, C5.1, C6.1, C7.1, C8.1, C9.1, U10.10 (2I0), U10.6 (1I0), U11.10 (2I0), U11.6 (1I0), U12.10 (2I0), U12.6 (1I0), U25.10 (ENT), U25.7 (ENP), U25.9 (~{LOAD}), U32.16 (VCC), U33.16 (VCC), U34.16 (VCC), U35.16 (VCC), U36.16 (VCC), U37.16 (VCC), U38.16 (VCC), U39.16 (VCC), U40.16 (VCC), U41.16 (VCC), U42.20 (VCC), U43.16 (VCC), U44.16 (VCC), U45.16 (VCC), U46.16 (VCC), U48.16 (VCC), U50.16 (VCC), U51.16 (VCC), U52.16 (VCC), U53.16 (VCC), U54.16 (VCC), U55.16 (VCC), U56.16 (VCC), U57.27 (~{WE}), U57.28 (VCC), U58.27 (~{WE}), U58.28 (VCC), U59.28 (VCC), U60.28 (VCC), U61.24 (VCC), U62.4 (VDD), U63.14 (VCC)
- net A0: no longer U59.10 (A0), U61.8 (A0)
- net A1: no longer U59.9 (A1), U61.7 (A1)
- net A10: no longer U59.21 (A10), U61.19 (A10)
- net A11: no longer U59.23 (A11)
- net A12: no longer U59.2 (A12)
- net A14: no longer U59.1 (A14)
- net A2: no longer U59.8 (A2), U61.6 (A2)
- net A3: no longer U59.7 (A3), U61.5 (A3)
- net A4: no longer U59.6 (A4), U61.4 (A4)
- net A5: no longer U59.5 (A5), U61.3 (A5)
- net A6: no longer U59.4 (A6), U61.2 (A6)
- net A7: no longer U59.3 (A7), U61.1 (A7)
- net A8: no longer U59.25 (A8), U61.23 (A8)
- net A9: no longer U59.24 (A9), U61.22 (A9)
- net ALU_A0: now also U14.1 (1A), U16.1 (1A)
- net ALU_A0_2: no longer U1.3 (Q0)
- net ALU_A1: now also U14.4 (2A), U16.4 (2A)
- net ALU_A1_2: no longer U1.4 (Q1)
- net ALU_A2: now also U14.9 (3A), U16.9 (3A)
- net ALU_A2_2: no longer U1.5 (Q2)
- net ALU_A3: now also U14.12 (4A), U16.12 (4A)
- net ALU_A3_2: no longer U1.6 (Q3)
- net ALU_A4: now also U15.1 (1A), U17.1 (1A)
- net ALU_A4_2: no longer U3.3 (Q0)
- net ALU_A5: now also U15.4 (2A), U17.4 (2A)
- net ALU_A5_2: no longer U3.4 (Q1)
- net ALU_A6: now also U15.9 (3A), U17.9 (3A)
- net ALU_A6_2: no longer U3.5 (Q2)
- net ALU_A7: now also U15.12 (4A), U17.12 (4A)
- net ALU_A7_2: no longer U3.6 (Q3)
- net ALU_B0: now also U14.2 (1B), U16.2 (1B), U38.3 (1I3), U7.3 (1Y); no longer U33.3 (Q0)
- net ALU_B0_2: no longer U2.3 (Q0)
- net ALU_B1: now also U14.5 (2B), U16.5 (2B), U38.13 (2I3), U7.6 (2Y); no longer U33.4 (Q1)
- net ALU_B1_2: no longer U2.4 (Q1)
- net ALU_B2: now also U14.10 (3B), U16.10 (3B), U39.3 (1I3), U7.8 (3Y); no longer U33.5 (Q2)
- net ALU_B2_2: no longer U2.5 (Q2)
- net ALU_B3: now also U14.13 (4B), U16.13 (4B), U39.13 (2I3), U7.11 (4Y); no longer U33.6 (Q3)
- net ALU_B3_2: no longer U2.6 (Q3)
- net ALU_B4: now also U15.2 (1B), U17.2 (1B), U40.3 (1I3), U8.3 (1Y); no longer U35.3 (Q0)
- net ALU_B4_2: no longer U4.3 (Q0)
- net ALU_B5: now also U15.5 (2B), U17.5 (2B), U40.13 (2I3), U8.6 (2Y); no longer U35.4 (Q1)
- net ALU_B5_2: no longer U4.4 (Q1)
- net ALU_B6: now also U15.10 (3B), U17.10 (3B), U41.3 (1I3), U8.8 (3Y); no longer U35.5 (Q2)
- net ALU_B6_2: no longer U4.5 (Q2)
- net ALU_B7: now also U15.13 (4B), U17.13 (4B), U41.13 (2I3), U8.11 (4Y); no longer U35.6 (Q3)
- net ALU_B7_2: no longer U4.6 (Q3)
- net ALU_MUX_OUT0: now also U18.1 (1A)
- net ALU_MUX_OUT1: now also U18.2 (1B)
- net ALU_MUX_OUT2: now also U18.4 (2A)
- net ALU_MUX_OUT3: now also U18.5 (2B)
- net ALU_MUX_OUT4: now also U18.9 (3A)
- net ALU_MUX_OUT5: now also U18.10 (3B)
- net ALU_MUX_OUT6: now also U18.12 (4A)
- net ALU_MUX_OUT7: now also U18.13 (4B)
- net ALU_S1: now also U38.10 (2I0); no longer U38.5 (1I1)
- net ALU_S2: now also U39.6 (1I0); no longer U38.4 (1I2)
- net ALU_S3: now also U39.10 (2I0); no longer U38.3 (1I3)
- net ALU_S4: now also U40.6 (1I0); no longer U39.6 (1I0)
- net ALU_S5: now also U40.10 (2I0); no longer U39.5 (1I1)
- net ALU_S6: now also U41.6 (1I0); no longer U39.4 (1I2)
- net ALU_S7: now also U41.10 (2I0); no longer U39.3 (1I3)
- net CLK: now also U1.7 (CP), U2.7 (CP), U25.2 (CLK), U3.7 (CP), U4.7 (CP)
- net CLK_2: no longer U1.7 (CP), U2.7 (CP), U25.2 (CLK), U3.7 (CP), U4.7 (CP)
- net D0: no longer U59.11 (I/O0)
- net D1: no longer U59.12 (I/O1)
- net D2: no longer U59.13 (I/O2)
- net D3: no longer U59.15 (I/O3)
- net DBUS0: now also U1.14 (D0), U3.14 (D0), U44.3 (Q0), U46.3 (Q0), U48.3 (Q0), U50.3 (Q0); no longer U34.14 (D0), U35.14 (D0), U45.14 (D0), U47.14 (D0), U49.14 (D0), U51.14 (D0), U56.14 (D0)
- net DBUS0_2: no longer U1.14 (D0), U2.14 (D0), U3.14 (D0), U4.14 (D0)
- net DBUS1: now also U1.13 (D1), U3.13 (D1), U44.4 (Q1), U46.4 (Q1), U48.4 (Q1), U50.4 (Q1); no longer U34.13 (D1), U35.13 (D1), U45.13 (D1), U47.13 (D1), U49.13 (D1), U51.13 (D1), U56.13 (D1)
- net DBUS1_2: no longer U1.13 (D1), U2.13 (D1), U3.13 (D1), U4.13 (D1)
- net DBUS2: now also U1.12 (D2), U3.12 (D2), U44.5 (Q2), U46.5 (Q2), U48.5 (Q2), U50.5 (Q2); no longer U34.12 (D2), U35.12 (D2), U45.12 (D2), U47.12 (D2), U49.12 (D2), U51.12 (D2), U56.12 (D2)
- net DBUS2_2: no longer U1.12 (D2), U2.12 (D2), U3.12 (D2), U4.12 (D2)
- net DBUS3: now also U1.11 (D3), U3.11 (D3), U44.6 (Q3), U46.6 (Q3), U48.6 (Q3), U50.6 (Q3); no longer U34.11 (D3), U35.11 (D3), U45.11 (D3), U47.11 (D3), U49.11 (D3), U51.11 (D3), U56.11 (D3)
- net DBUS3_2: no longer U1.11 (D3), U2.11 (D3), U3.11 (D3), U4.11 (D3)
- net DBUS4: now also U2.14 (D0), U34.14 (D0), U35.14 (D0), U45.14 (D0), U45.3 (Q0), U47.14 (D0), U47.3 (Q0), U49.14 (D0), U49.3 (Q0), U51.14 (D0), U51.3 (Q0), U56.14 (D0)
- net DBUS5: now also U2.13 (D1), U34.13 (D1), U35.13 (D1), U45.13 (D1), U45.4 (Q1), U47.13 (D1), U47.4 (Q1), U49.13 (D1), U49.4 (Q1), U51.13 (D1), U51.4 (Q1), U56.13 (D1)
- net DBUS6: now also U2.12 (D2), U34.12 (D2), U35.12 (D2), U45.12 (D2), U45.5 (Q2), U47.12 (D2), U47.5 (Q2), U49.12 (D2), U49.5 (Q2), U51.12 (D2), U51.5 (Q2), U56.12 (D2)
- net DBUS7: now also U2.11 (D3), U34.11 (D3), U35.11 (D3), U45.11 (D3), U45.6 (Q3), U47.11 (D3), U47.6 (Q3), U49.11 (D3), U49.6 (Q3), U51.11 (D3), U51.6 (Q3), U56.11 (D3)
- net GND: now also U1.1 (#OE1), U1.2 (#OE), U10.1 (~{1E}), U10.11 (2I1), U10.15 (~{2E}), U10.2 (S1), U10.5 (1I1), U11.1 (~{1E}), U11.11 (2I1), U11.15 (~{2E}), U11.2 (S1), U11.5 (1I1), U12.1 (~{1E}), U12.11 (2I1), U12.15 (~{2E}), U12.2 (S1), U12.5 (1I1), U2.1 (#OE1), U2.2 (#OE), U25.3 (A), U25.4 (B), U25.5 (C), U25.6 (D), U3.1 (#OE1), U3.2 (#OE), U4.1 (#OE1), U4.11 (D3), U4.12 (D2), U4.2 (#OE), U43.1 (~{1E}), U57.1 (A14), U57.2 (A12), U57.21 (A10), U57.23 (A11), U57.24 (A9), U57.26 (A13), U58.1 (A14), U58.2 (A12), U58.21 (A10), U58.23 (A11), U58.24 (A9), U58.26 (A13), U59.1 (A14), U59.2 (A12), U59.21 (A10), U59.23 (A11), U59.24 (A9), U59.26 (A13), U9.1 (~{1E}), U9.15 (~{2E}), U9.2 (S1); no longer U36.7 (CIN), U52.10 (ENT), U52.7 (ENP), U60.22 (~{OE})
- net REG_SEL0: now also U9.7 (1Y); no longer U55.3 (Q0)
- net REG_SEL1: now also U9.9 (2Y); no longer U55.4 (Q1)
- net RESET_N: now also U25.1 (~{CLR})
- net ALU_AND7: now reaches U41.11 (2I1)
- net ALU_AND7: now also U15.11 (4Y)
- net ALU_OR7: now reaches U41.12 (2I2)
- net ALU_OR7: now also U17.11 (4Y)
- net ALU_SEL0: now reaches U41.14 (S0)
- net ALU_SEL0: now also U38.14 (S0), U39.14 (S0), U40.14 (S0), U58.17 (I/O5)
- net ALU_SEL1: now reaches U41.2 (S1)
- net ALU_SEL1: now also U38.2 (S1), U39.2 (S1), U40.2 (S1), U58.18 (I/O6)
- net ALU_OR6: now reaches U41.4 (1I2)
- net ALU_OR6: now also U17.8 (3Y)
- net ALU_AND6: now reaches U41.5 (1I1)
- net ALU_AND6: now also U15.8 (3Y)
- net MARL0: now reaches U52.3 (A)
- net MARL0: now also U1.3 (Q0), U61.8 (A0)
- net MARL1: now reaches U52.4 (B)
- net MARL1: now also U1.4 (Q1), U61.7 (A1)
- net MARL2: now reaches U52.5 (C)
- net MARL2: now also U1.5 (Q2), U61.6 (A2)
- net MARL3: now reaches U52.6 (D)
- net MARL3: now also U1.6 (Q3), U61.5 (A3)
- net PC_LOAD_N: now reaches U52.9 (~{LOAD})
- net PC_LOAD_N: now also U20.12 (6Y), U53.9 (~{LOAD}), U54.9 (~{LOAD})
- net ALU_B_RAW0: now reaches U7.1 (1A)
- net ALU_B_RAW0: now also U33.3 (Q0)
- net SU: now reaches U7.10 (3B)
- net SU: now also U36.7 (CIN), U58.19 (I/O7), U7.13 (4B), U7.2 (1B), U7.5 (2B), U8.10 (3B), U8.13 (4B), U8.2 (1B), U8.5 (2B)
- net ALU_B_RAW3: now reaches U7.12 (4A)
- net ALU_B_RAW3: now also U33.6 (Q3)
- net ALU_B_RAW1: now reaches U7.4 (2A)
- net ALU_B_RAW1: now also U33.4 (Q1)
- net ALU_B_RAW2: now reaches U7.9 (3A)
- net ALU_B_RAW2: now also U33.5 (Q2)
- net ALU_AND3: now reaches U14.11 (4Y)
- net ALU_AND3: now also U39.11 (2I1)
- net ALU_AND0: now reaches U14.3 (1Y)
- net ALU_AND0: now also U38.5 (1I1)
- net ALU_AND1: now reaches U14.6 (2Y)
- net ALU_AND1: now also U38.11 (2I1)
- net ALU_AND2: now reaches U14.8 (3Y)
- net ALU_AND2: now also U39.5 (1I1)
- net ZT_G1: now reaches U19.1 (1A)
- net ZT_G1: now also U18.3 (1Y)
- net ZT_G6: now reaches U19.10 (3B)
- net ZT_G6: now also U19.6 (2Y)
- net FI_OR: now reaches U19.11 (4Y)
- net FI_OR: now also U11.14 (S0)
- net FI_ZN: now reaches U19.12 (4A)
- net FI_ZN: now also U59.12 (I/O1)
- net FI_C: now reaches U19.13 (4B)
- net FI_C: now also U59.13 (I/O2)
- net ZT_G2: now reaches U19.2 (1B)
- net ZT_G2: now also U18.6 (2Y)
- net ZT_G5: now reaches U19.3 (1Y)
- net ZT_G5: now also U19.9 (3A)
- net ZT_G3: now reaches U19.4 (2A)
- net ZT_G3: now also U18.8 (3Y)
- net ZT_G4: now reaches U19.5 (2B)
- net ZT_G4: now also U18.11 (4Y)
- net ZT_G7: now reaches U19.8 (3Y)
- net ZT_G7: now also U10.14 (S0)
- net REGSEL_Y0: now reaches U43.4 (~{1Y0})
- net REGSEL_Y0: now also U44.1 (#OE1), U44.9 (#E1), U45.1 (#OE1), U45.9 (#E1)
- net REGSEL_Y1: now reaches U43.5 (~{1Y1})
- net REGSEL_Y1: now also U46.1 (#OE1), U46.9 (#E1), U47.1 (#OE1), U47.9 (#E1)
- net REGSEL_Y2: now reaches U43.6 (~{1Y2})
- net REGSEL_Y2: now also U48.1 (#OE1), U48.9 (#E1), U49.1 (#OE1), U49.9 (#E1)
- net REGSEL_Y3: now reaches U43.7 (~{1Y3})
- net REGSEL_Y3: now also U50.1 (#OE1), U50.9 (#E1), U51.1 (#OE1), U51.9 (#E1)
- net MAR_LOW_IN: now reaches U2.10 (#E2)
- net MAR_LOW_IN: now also U1.10 (#E2), U1.9 (#E1), U2.9 (#E1), U57.16 (I/O4)
- net IR_RD1: now reaches U9.10 (2I0)
- net IR_RD1: now also U55.6 (Q3)
- net IR_RS1: now reaches U9.11 (2I1)
- net IR_RS1: now also U55.4 (Q1)
- net RS_SEL: now reaches U9.14 (S0)
- net RS_SEL: now also U58.11 (I/O0)
- net IR_RS0: now reaches U9.5 (1I1)
- net IR_RS0: now also U55.3 (Q0)
- net IR_RD0: now reaches U9.6 (1I0)
- net IR_RD0: now also U55.5 (Q2)
- net REG_IN_N: now reaches U44.10 (#E2)
- net REG_IN_N: now also U20.8 (4Y), U45.10 (#E2), U46.10 (#E2), U47.10 (#E2), U48.10 (#E2), U49.10 (#E2), U50.10 (#E2), U51.10 (#E2)
- net REG_OUT_N: now reaches U44.2 (#OE)
- net REG_OUT_N: now also U20.10 (5Y), U45.2 (#OE), U46.2 (#OE), U47.2 (#OE), U48.2 (#OE), U49.2 (#OE), U50.2 (#OE), U51.2 (#OE)
- net STEP2: now reaches U25.12 (QC)
- net STEP2: now also U57.6 (A4), U58.6 (A4), U59.6 (A4)
- net STEP1: now reaches U25.13 (QB)
- net STEP1: now also U57.7 (A3), U58.7 (A3), U59.7 (A3)
- net STEP0: now reaches U25.14 (QA)
- net STEP0: now also U57.8 (A2), U58.8 (A2), U59.8 (A2)
- net ALU_B_RAW4: now reaches U8.1 (1A)
- net ALU_B_RAW4: now also U35.3 (Q0)
- net ALU_B_RAW7: now reaches U8.12 (4A)
- net ALU_B_RAW7: now also U35.6 (Q3)
- net ALU_B_RAW5: now reaches U8.4 (2A)
- net ALU_B_RAW5: now also U35.4 (Q1)
- net ALU_B_RAW6: now reaches U8.9 (3A)
- net ALU_B_RAW6: now also U35.5 (Q2)
- net Z_COMPUTED: now reaches U10.7 (1Y)
- net Z_COMPUTED: now also U10.9 (2Y), U4.14 (D0)
- net MAR_HIGH_IN: now reaches U3.10 (#E2)
- net MAR_HIGH_IN: now also U3.9 (#E1), U57.17 (I/O5)
- net C: now reaches U58.10 (A0)
- net C: now also U4.4 (Q1), U57.10 (A0), U59.10 (A0)
- net REG_IN: now reaches U58.12 (I/O1)
- net REG_IN: now also U20.9 (4A)
- net REG_OUT: now reaches U58.13 (I/O2)
- net REG_OUT: now also U20.11 (5A)
- net A_IN: now reaches U58.15 (I/O3)
- net A_IN: now also U32.10 (#E2), U32.9 (#E1), U34.10 (#E2), U34.9 (#E1)
- net TEMP_IN: now reaches U58.16 (I/O4)
- net TEMP_IN: now also U33.10 (#E2), U33.9 (#E1), U35.10 (#E2), U35.9 (#E1)
- net OPCODE3: now reaches U58.25 (A8)
- net OPCODE3: now also U56.6 (Q3), U57.25 (A8), U59.25 (A8)
- net OPCODE2: now reaches U58.3 (A7)
- net OPCODE2: now also U56.5 (Q2), U57.3 (A7), U59.3 (A7)
- net OPCODE1: now reaches U58.4 (A6)
- net OPCODE1: now also U56.4 (Q1), U57.4 (A6), U59.4 (A6)
- net OPCODE0: now reaches U58.5 (A5)
- net OPCODE0: now also U56.3 (Q0), U57.5 (A5), U59.5 (A5)
- net Z: now reaches U58.9 (A1)
- net Z: now also U4.3 (Q0), U57.9 (A1), U59.9 (A1)
- net ALU_AND5: now reaches U40.11 (2I1)
- net ALU_AND5: now also U15.6 (2Y)
- net ALU_OR5: now reaches U40.12 (2I2)
- net ALU_OR5: now also U17.6 (2Y)
- net ALU_OR4: now reaches U40.4 (1I2)
- net ALU_OR4: now also U17.3 (1Y)
- net ALU_AND4: now reaches U40.5 (1I1)
- net ALU_AND4: now also U15.3 (1Y)
- net C_COMPUTED: now reaches U37.9 (COUT)
- net C_COMPUTED: now also U4.13 (D1)
- net IR_IN: now reaches U56.10 (#E2)
- net IR_IN: now also U55.10 (#E2), U55.9 (#E1), U56.9 (#E1), U57.15 (I/O3)
- net FI_LATCH_N: now reaches U4.10 (#E2)
- net FI_LATCH_N: now also U11.7 (1Y), U11.9 (2Y), U4.9 (#E1)
- net MARL4: now reaches U53.3 (A)
- net MARL4: now also U2.3 (Q0), U61.4 (A4)
- net MARL5: now reaches U53.4 (B)
- net MARL5: now also U2.4 (Q1), U61.3 (A5)
- net MARL6: now reaches U53.5 (C)
- net MARL6: now also U2.5 (Q2), U61.2 (A6)
- net MARL7: now reaches U53.6 (D)
- net MARL7: now also U2.6 (Q3), U61.1 (A7)
- net MARH0: now reaches U54.3 (A)
- net MARH0: now also U3.3 (Q0), U61.23 (A8)
- net MARH1: now reaches U54.4 (B)
- net MARH1: now also U3.4 (Q1), U61.22 (A9)
- net MARH2: now reaches U54.5 (C)
- net MARH2: now also U3.5 (Q2), U61.19 (A10)
- net MARH3: now reaches U54.6 (D)
- net MARH3: now also U3.6 (Q3)
- net ALU_OR1: now reaches U38.12 (2I2)
- net ALU_OR1: now also U16.6 (2Y)
- net EO_N: now reaches U42.19 (~{OE})
- net EO_N: now also U12.7 (1Y), U12.9 (2Y)
- net IROM_OUT: now reaches U57.11 (I/O0)
- net IROM_OUT: now also U20.1 (1A)
- net RAM_OUT: now reaches U57.12 (I/O1)
- net RAM_OUT: now also U20.3 (2A)
- net RAM_IN: now reaches U57.13 (I/O2)
- net RAM_IN: now also U20.5 (3A)
- net PC_INC: now reaches U57.18 (I/O6)
- net PC_INC: now also U52.10 (ENT), U52.7 (ENP)
- net PC_LOAD: now reaches U57.19 (I/O7)
- net PC_LOAD: now also U20.13 (6A)
- net ALU_OR3: now reaches U16.11 (4Y)
- net ALU_OR3: now also U39.12 (2I2)
- net ALU_OR0: now reaches U16.3 (1Y)
- net ALU_OR0: now also U38.4 (1I2)
- net ALU_OR2: now reaches U16.8 (3Y)
- net ALU_OR2: now also U39.4 (1I2)
- net IROM_OUT_N: now reaches U20.2 (1Y)
- net IROM_OUT_N: now also U60.22 (~{OE})
- net RAM_OUT_N: now reaches U20.4 (2Y)
- net RAM_IN_N: now reaches U20.6 (3Y)
- net EO: now reaches U12.14 (S0)
- net EO: now also U59.11 (I/O0)
- removed net ALU_LOAD_HIGH: U34.10 (#E2), U34.9 (#E1), U35.10 (#E2), U35.9 (#E1)
- removed net ALU_LOAD_LOW: U32.10 (#E2), U32.9 (#E1), U33.10 (#E2), U33.9 (#E1)
- new net HLT: U59.15 (I/O3)
